File: hbkb.kicad_pcb (KiCad board)
At the start: 2 copper layers, 317.5 x 139.7 mm, 128 parts, among them J1 Conn_01x07, J2 Conn_01x04, J3 Conn_01x03, J4 Conn_01x07

Commit message: add shift register
Parts:
- added J5: Conn_01x05, Connector_PinHeader_2.54mm:PinHeader_1x05_P2.54mm_Vertical, F.Cu at (172.7, 124.1)
- added U1: 74HC595, Package_DIP:DIP-16_W7.62mm, F.Cu at (76.5, 146.4)
- added U2: 74HC595, Package_DIP:DIP-16_W7.62mm, F.Cu at (170.2, 148.2)
- added U3: 74HC595, Package_DIP:DIP-16_W7.62mm, F.Cu at (272.2, 165.5)
- moved J2 153.1 mm to (164.7, 131.8)
- moved J3 137.5 mm to (174.9, 48.1), turned to 270 degrees
- moved J4 25.1 mm to (220.3, 47.0)
- moved D21 8.89 mm to (141.0, 106.9), turned to 345 degrees
- moved D27 8.88 mm to (291.6, 84.2), turned to 15 degrees
- moved D11 8.22 mm to (247.9, 68.4), turned to 15 degrees
- moved D19 8.20 mm to (105.0, 93.5), turned to 345 degrees
- moved D24 8.00 mm to (235.3, 95.2), turned to 15 degrees
- moved D55 7.45 mm to (301.5, 121.0), turned to 15 degrees
- moved D46 7.45 mm to (77.7, 121.8), turned to 345 degrees
- moved D66 7.27 mm to (197.1, 172.0), turned to 15 degrees
- moved D36 7.17 mm to (204.7, 127.3), turned to 15 degrees
- moved D14 6.94 mm to (304.9, 60.9), turned to 15 degrees
- moved D6 6.87 mm to (127.8, 83.4), turned to 345 degrees
- moved D9 6.82 mm to (213.1, 85.6), turned to 15 degrees
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Connections:
- net /KeyscanMatrix/COL1 renamed /COL1
- net /KeyscanMatrix/COL10 renamed /COL10
- net /KeyscanMatrix/COL11 renamed /COL11
- net /KeyscanMatrix/COL12 renamed /COL12
- net /KeyscanMatrix/COL13 renamed /COL13
- net /KeyscanMatrix/COL14 renamed /COL14
- net /KeyscanMatrix/COL15 renamed /COL15
- net /KeyscanMatrix/COL16 renamed /COL16
- net /KeyscanMatrix/COL17 renamed /COL17
- net /KeyscanMatrix/COL2 renamed /COL2
- net /KeyscanMatrix/COL3 renamed /COL3
- net /KeyscanMatrix/COL4 renamed /COL4
- net /KeyscanMatrix/COL5 renamed /COL5
- net /KeyscanMatrix/COL6 renamed /COL6
- net /KeyscanMatrix/COL7 renamed /COL7
- net /KeyscanMatrix/COL8 renamed /COL8
- net /KeyscanMatrix/COL9 renamed /COL9
Other:
- board text added: "HebiKeyboard v1.0"

Commit message: finish matrix routing, moving from 4 rows to 5 rows
Parts:
- U1, U3: moved to B.Cu
- moved J5 84.7 mm to (90.4, 144.1)
- moved J2 32.0 mm to (169.4, 100.2)
- moved U2 27.8 mm to (172.8, 175.9)
- moved U3 20.0 mm to (273.1, 145.5), turned to 285 degrees
- moved U1 18.8 mm to (58.0, 142.6), turned to 255 degrees
- moved D48 7.82 mm to (120.1, 140.7), turned to 165 degrees
- moved D29 7.80 mm to (33.0, 97.7), turned to 165 degrees
- moved D52 7.78 mm to (245.2, 132.2), turned to 15 degrees
- moved D7 7.76 mm to (153.4, 90.4), turned to 165 degrees
- moved D18 7.73 mm to (95.1, 86.7), turned to 165 degrees
- moved D19 7.73 mm to (112.5, 95.4), turned to 165 degrees
- moved D33 7.73 mm to (107.6, 113.7), turned to 165 degrees
- moved D16 7.73 mm to (56.3, 84.3), turned to 165 degrees
- moved D2 7.73 mm to (61.2, 65.8), turned to 165 degrees
- moved D43 7.73 mm to (28.1, 116.2), turned to 165 degrees
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Connections:
- J5 pad 1: /OE -> /SER
- J5 pad 2: /RCLK -> /OE
- J5 pad 3: /SRCLR -> /RCLK
- J5 pad 5: Net-(J5-Pad5) -> /SRCLR
- S32 pad 1: Net-(S32-Pad1) -> /KeyscanMatrix/ROW3
- S33 pad 1: Net-(S32-Pad1) -> /KeyscanMatrix/ROW3
- S34 pad 1: Net-(S32-Pad1) -> /KeyscanMatrix/ROW3
- S35 pad 1: Net-(S32-Pad1) -> /KeyscanMatrix/ROW3
- U1 pad 14: Net-(J5-Pad5) -> /SER
Routing:
- net /COL17: track 0.00 -> 193.0 mm
- net /COL1: track 0.00 -> 191.7 mm
- net /COL7: track 0.00 -> 173.6 mm
- net /COL11: track 0.00 -> 172.7 mm
- net /COL16: track 0.00 -> 162.6 mm
- net /COL2: track 0.00 -> 155.9 mm
- net /KeyscanMatrix/ROW4: track 0.00 -> 155.5 mm
- net /KeyscanMatrix/ROW1: track 0.00 -> 155.3 mm
- net /COL6: track 0.00 -> 142.8 mm
- net /COL12: track 0.00 -> 135.8 mm
- net /COL15: track 0.00 -> 132.8 mm
- net /COL3: track 0.00 -> 130.4 mm
- net /COL5: track 0.00 -> 119.3 mm
- net /COL4: track 0.00 -> 118.4 mm
- net Net-(S22-Pad1): track 0.00 -> 117.4 mm
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
Commit message: finish entire board
Parts:
- removed J5: Conn_01x05, Connector_PinHeader_2.54mm:PinHeader_1x05_P2.54mm_Vertical
- removed U2: 74HC595, Package_DIP:DIP-16_W7.62mm
- J2: value Conn_01x04 -> Conn_01x05; footprint Connector_PinHeader_2.54mm:PinHeader_1x04_P2.54mm_Vertical -> Connector_PinHeader_2.54mm:PinHeader_1x05_P2.54mm_Vertical
- J3: value Conn_01x03 -> Conn_01x07; footprint Connector_PinHeader_2.54mm:PinHeader_1x03_P2.54mm_Vertical -> Connector_PinHeader_2.54mm:PinHeader_1x07_P2.54mm_Vertical
- moved J3 85.7 mm to (173.0, 133.9), turned to 0 degrees
- moved J2 14.4 mm to (172.7, 114.2), turned to 0 degrees
Connections:
- D10 pad 2: /COL13 -> /COL10
- D11 pad 2: /COL14 -> /COL11
- D12 pad 2: /COL15 -> /COL12
- D13 pad 2: /COL16 -> /COL13
- D14 pad 2: /COL17 -> /COL14
- D22 pad 2: /COL11 -> /COL8
- D23 pad 2: /COL12 -> /COL9
- D24 pad 2: /COL13 -> /COL10
- D25 pad 2: /COL14 -> /COL11
- D26 pad 2: /COL15 -> /COL12
- D27 pad 2: /COL16 -> /COL13
- D28 pad 2: /COL17 -> /COL14
- D36 pad 2: /COL11 -> /COL8
- D37 pad 2: /COL12 -> /COL9
- D38 pad 2: /COL13 -> /COL10
- D39 pad 2: /COL14 -> /COL11
- D40 pad 2: /COL15 -> /COL12
- D41 pad 2: /COL16 -> /COL13
- D42 pad 2: /COL17 -> /COL14
- D50 pad 2: /COL11 -> /COL8
- D51 pad 2: /COL12 -> /COL9
- D52 pad 2: /COL13 -> /COL10
- D53 pad 2: /COL14 -> /COL11
- D54 pad 2: /COL15 -> /COL12
- D55 pad 2: /COL16 -> /COL13
- D56 pad 2: /COL17 -> /COL14
- D57 pad 2: /COL8 -> /COL3
- D58 pad 2: /COL9 -> /COL4
- D59 pad 2: /COL10 -> /COL5
- D66 pad 2: /COL8 -> /COL10
- D67 pad 2: /COL9 -> /COL11
- D68 pad 2: /COL10 -> /COL12
- D8 pad 2: /COL11 -> /COL8
- D9 pad 2: /COL12 -> /COL9
- J2 pad 1: /KeyscanMatrix/ROW4 -> /KeyscanMatrix/ROW1
- J2 pad 2: /KeyscanMatrix/ROW3 -> /KeyscanMatrix/ROW2
- J2 pad 3: /KeyscanMatrix/ROW2 -> /KeyscanMatrix/ROW3
- J2 pad 4: /KeyscanMatrix/ROW1 -> /KeyscanMatrix/ROW4
- J3 pad 1: /COL8 -> /SER
- J3 pad 2: /COL9 -> /OE
- J3 pad 3: /COL10 -> /RCLK
- J4 pad 1: /COL11 -> /COL8
- J4 pad 2: /COL12 -> /COL9
- J4 pad 3: /COL13 -> /COL10
- J4 pad 4: /COL14 -> /COL11
- J4 pad 5: /COL15 -> /COL12
- J4 pad 6: /COL16 -> /COL13
- J4 pad 7: /COL17 -> /COL14
- S10 pad 1: Net-(S10-Pad1) -> /KeyscanMatrix/ROW1
- S11 pad 1: Net-(S10-Pad1) -> /KeyscanMatrix/ROW1
- S12 pad 1: Net-(S10-Pad1) -> /KeyscanMatrix/ROW1
- S13 pad 1: Net-(S10-Pad1) -> /KeyscanMatrix/ROW1
- S14 pad 1: Net-(S10-Pad1) -> /KeyscanMatrix/ROW1
- S22 pad 1: Net-(S22-Pad1) -> /KeyscanMatrix/ROW2
- S23 pad 1: Net-(S22-Pad1) -> /KeyscanMatrix/ROW2
- S24 pad 1: Net-(S22-Pad1) -> /KeyscanMatrix/ROW2
- S25 pad 1: Net-(S22-Pad1) -> /KeyscanMatrix/ROW2
- S26 pad 1: Net-(S22-Pad1) -> /KeyscanMatrix/ROW2
- S27 pad 1: Net-(S22-Pad1) -> /KeyscanMatrix/ROW2
- S28 pad 1: Net-(S22-Pad1) -> /KeyscanMatrix/ROW2
- S36 pad 1: Net-(S36-Pad1) -> /KeyscanMatrix/ROW3
- S37 pad 1: Net-(S36-Pad1) -> /KeyscanMatrix/ROW3
- S38 pad 1: Net-(S36-Pad1) -> /KeyscanMatrix/ROW3
- S39 pad 1: Net-(S36-Pad1) -> /KeyscanMatrix/ROW3
- S40 pad 1: Net-(S36-Pad1) -> /KeyscanMatrix/ROW3
- S41 pad 1: Net-(S36-Pad1) -> /KeyscanMatrix/ROW3
- S42 pad 1: Net-(S36-Pad1) -> /KeyscanMatrix/ROW3
- S50 pad 1: Net-(S50-Pad1) -> /KeyscanMatrix/ROW4
- S51 pad 1: Net-(S50-Pad1) -> /KeyscanMatrix/ROW4
- S52 pad 1: Net-(S50-Pad1) -> /KeyscanMatrix/ROW4
- S53 pad 1: Net-(S50-Pad1) -> /KeyscanMatrix/ROW4
- S54 pad 1: Net-(S50-Pad1) -> /KeyscanMatrix/ROW4
- S55 pad 1: Net-(S50-Pad1) -> /KeyscanMatrix/ROW4
- S56 pad 1: Net-(S50-Pad1) -> /KeyscanMatrix/ROW4
- S57 pad 1: /KeyscanMatrix/ROW1 -> /KeyscanMatrix/ROW5
- S58 pad 1: /KeyscanMatrix/ROW1 -> /KeyscanMatrix/ROW5
- S59 pad 1: /KeyscanMatrix/ROW1 -> /KeyscanMatrix/ROW5
- S66 pad 1: /KeyscanMatrix/ROW4 -> /KeyscanMatrix/ROW5
- S67 pad 1: /KeyscanMatrix/ROW4 -> /KeyscanMatrix/ROW5
- S68 pad 1: /KeyscanMatrix/ROW4 -> /KeyscanMatrix/ROW5
- S8 pad 1: Net-(S10-Pad1) -> /KeyscanMatrix/ROW1
- S9 pad 1: Net-(S10-Pad1) -> /KeyscanMatrix/ROW1
- U3 pad 1: /COL12 -> /COL9
- U3 pad 14: Net-(U2-Pad9) -> Net-(U1-Pad9)
- U3 pad 15: /COL11 -> /COL8
- U3 pad 2: /COL13 -> /COL10
- U3 pad 3: /COL14 -> /COL11
- U3 pad 4: /COL15 -> /COL12
- U3 pad 5: /COL16 -> /COL13
- U3 pad 6: /COL17 -> /COL14
Routing:
- net /OE: track 0.00 -> 238.0 mm, vias 0 -> 2
- net /RCLK: track 0.00 -> 237.5 mm, vias 0 -> 2
- net /SRCLK: track 0.00 -> 236.0 mm, vias 0 -> 2
- net /SRCLR: track 0.00 -> 235.9 mm, vias 0 -> 2
- net Net-(U1-Pad9): track 0.00 -> 215.1 mm, vias 0 -> 3
- net /KeyscanMatrix/ROW5: track 0.00 -> 200.4 mm
- net /COL17: track 193.0 -> 0.00 mm
- net /KeyscanMatrix/ROW2: track 117.0 -> 294.8 mm
- net /COL10: track 0.00 -> 177.7 mm, vias 0 -> 1
- net /COL8: track 0.00 -> 172.7 mm
- net /KeyscanMatrix/ROW3: track 117.3 -> 285.5 mm
- net /KeyscanMatrix/ROW1: track 155.3 -> 319.9 mm
- net /COL16: track 162.6 -> 0.00 mm
- net /KeyscanMatrix/ROW4: track 155.5 -> 300.8 mm
- net /COL9: track 0.00 -> 135.8 mm
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- added copper zone on F.Cu, net +5V
- added copper zone on B.Cu, net GND

Commit message: entire copper fill
Parts:
- added REF**: MountingHole_3.2mm_M3, MountingHole:MountingHole_3.2mm_M3, F.Cu at (161.3, 63.5)
- added REF**: MountingHole_3.2mm_M3, MountingHole:MountingHole_3.2mm_M3, F.Cu at (21.6, 50.8)
- added REF**: MountingHole_3.2mm_M3, MountingHole:MountingHole_3.2mm_M3, F.Cu at (186.7, 63.5)
- added REF**: MountingHole_3.2mm_M3, MountingHole:MountingHole_3.2mm_M3, F.Cu at (199.4, 50.8)
- added REF**: MountingHole_3.2mm_M3, MountingHole:MountingHole_3.2mm_M3, F.Cu at (148.6, 50.8)
- added REF**: MountingHole_3.2mm_M3, MountingHole:MountingHole_3.2mm_M3, F.Cu at (174.0, 101.6)
- added REF**: MountingHole_3.2mm_M3, MountingHole:MountingHole_3.2mm_M3, F.Cu at (326.4, 152.4)
- added REF**: MountingHole_3.2mm_M3, MountingHole:MountingHole_3.2mm_M3, F.Cu at (326.4, 50.8)
- added REF**: MountingHole_3.2mm_M3, MountingHole:MountingHole_3.2mm_M3, F.Cu at (174.0, 50.8)
- added REF**: MountingHole_3.2mm_M3, MountingHole:MountingHole_3.2mm_M3, F.Cu at (21.6, 152.4)
Routing:
- net /COL6: track 142.8 -> 144.2 mm, vias 0 -> 1
- net /COL11: track 181.7 -> 182.8 mm
- net /COL12: track 200.6 -> 199.9 mm
- net /COL5: vias 2 -> 3
- net /COL4: vias 2 -> 3
Other:
- outline, holes or cut-outs redrawn
- board text added: "COL1"
- board text added: "COL14"
- board text added: "COL7"
- board text added: "COL8"
- board text added: "GND"
- board text added: "OE"
- board text added: "RCLK"
- board text added: "ROW1"
- board text added: "ROW5"
- board text added: "SER"
- board text added: "SRCLK"
- board text added: "SRCLR"
- board text added: "VCC"

Commit message: adjust bottom row position
Parts:
- removed REF** (x10): MountingHole_3.2mm_M3, MountingHole:MountingHole_3.2mm_M3
- moved D67 37.9 mm to (251.3, 154.6)
- moved S68 37.9 mm to (264.9, 140.8)
- moved D57 37.9 mm to (78.2, 149.6)
- moved D58 37.9 mm to (96.6, 154.6)
- moved D59 37.9 mm to (115.1, 159.5)
- moved D66 37.9 mm to (232.9, 159.5)
- moved D68 37.9 mm to (269.6, 149.7)
- moved S57 37.9 mm to (83.1, 140.8)
- moved S58 37.9 mm to (101.3, 145.8)
- moved S59 37.9 mm to (119.8, 150.6)
- moved S66 37.9 mm to (228.2, 150.7)
- moved S67 37.9 mm to (246.5, 145.8)
- moved U1 18.3 mm to (42.2, 151.6)
- moved U3 13.3 mm to (276.6, 158.2)
Routing:
- net +5V: track 36.0 -> 255.4 mm, vias 4 -> 2
- net /COL12: track 199.9 -> 137.9 mm
- net /KeyscanMatrix/ROW5: track 200.4 -> 250.3 mm, vias 0 -> 1
- net /COL11: track 182.8 -> 136.4 mm, vias 1 -> 0
- net /OE: track 238.0 -> 272.1 mm, vias 2 -> 0
- net /COL6: track 144.2 -> 176.2 mm, vias 1 -> 0
- net /COL3: track 193.9 -> 162.9 mm, vias 1 -> 0
- net /COL7: track 173.6 -> 204.2 mm
- net GND: track 0.00 -> 26.8 mm, vias 0 -> 1
- net /SER: track 118.0 -> 142.9 mm
- net /KeyscanMatrix/ROW2: track 294.8 -> 319.0 mm
- net /SRCLK: track 236.0 -> 257.4 mm, vias 2 -> 1
- net /SRCLR: track 235.9 -> 257.2 mm, vias 2 -> 0
- net /RCLK: track 237.5 -> 258.2 mm, vias 2 -> 1
- net /KeyscanMatrix/ROW4: track 300.8 -> 320.7 mm, vias 0 -> 1
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- added copper zone on F.Cu, net GND
- removed copper zone on F.Cu, net +5V
